File: Linear Power Supply - Summer 2024.kicad_sch (KiCad schematic)
At the start: 7 parts, among them IC1 LD1085V, T1 FP16-3000

Commit message: Big push on the PCB layout. I think ready to send to JLC or OSH...
Parts:
- C2: footprint (none) -> Chase's Footprints:Small Electrolytic Capacitor
- POT1: renamed from RV1; footprint (none) -> Potentiometer_THT:Potentiometer_ACP_CA14-H2,5_Horizontal
- R1: footprint (none) -> Resistor_THT:R_Axial_DIN0204_L3.6mm_D1.6mm_P7.62mm_Horizontal
Other:
- note added: "TO GND CHASSIS"
- company: Lotito Electric -> Lotito Laboratories
Changed lines of the file:
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@@
 	(title_block
 		(title "Linear Power Supply - SUMMER 2024")
-		(date "2024-06-08")
-		(company "Lotito Electric")
+		(date "2024-06-16")
+		(company "Lotito Laboratories")
 	)
 	(junction
@@
 	(wire
 		(pts
+			(xy 78.74 113.03) (xy 78.74 119.38)
+		)
+		(stroke
+			(width 0)
+			(type default)
+		)
+	)
+	(wire
+		(pts
 			(xy 78.74 87.63) (xy 93.98 87.63)
 		)
@@
 		(pts
 			(xy 125.73 76.2) (xy 125.73 85.09)
+		)
+		(stroke
+			(width 0)
+			(type default)
+		)
+	)
+	(wire
+		(pts
+			(xy 68.58 113.03) (xy 78.74 113.03)
 		)
 		(stroke
@@
 			(font
 				(size 1.27 1.27)
+			)
+		)
+	)
+	(text "TO GND CHASSIS"
+		(exclude_from_sim no)
+		(at 87.376 115.062 0)
+		(effects
+			(font
+				(face "JetBrainsMono NF")
+				(size 1.27 1.27)
+			)
+		)
+	)
+	(global_label "GND"
+		(shape input)
+		(at 68.58 113.03 180)
+		(fields_autoplaced yes)
+		(effects
+			(font
+				(size 1.27 1.27)
+			)
+			(justify right)
+		)
+		(property "Intersheetrefs" "${INTERSHEET_REFS}"
+			(at 62.6198 113.03 0)
+			(effects
+				(font
+					(size 1.27 1.27)
+				)
+				(justify right)
+				(hide yes)
 			)
 		)
@@
 			)
 		)
-		(property "Footprint" ""
+		(property "Footprint" "Chase's Footprints:Small Electrolytic Capacitor"
 			(at 210.82 97.79 0)
 			(effects
@@
 			)
 		)
-		(property "Footprint" ""
+		(property "Footprint" "Resistor_THT:R_Axial_DIN0204_L3.6mm_D1.6mm_P7.62mm_Horizontal"
 			(at 187.706 92.964 90)
 			(effects
@@
 		(dnp no)
 		(fields_autoplaced yes)
-		(property "Reference" "RV1"
+		(property "Reference" "POT1"
 			(at 170.18 110.4899 0)
 			(effects
@@
 			)
 		)
-		(property "Footprint" ""
+		(property "Footprint" "Potentiometer_THT:Potentiometer_ACP_CA14-H2,5_Horizontal"
 			(at 172.72 111.76 0)
 			(effects
@@
 			(project ""
 				(path "/1c8830c9-4fc6-4803-9490-280577e79dde"
-					(reference "RV1")
+					(reference "POT1")
 					(unit 1)
 				)
@@
 					(unit 1)
 				)
+			)
+		)
+	)
+	(symbol
+		(lib_id "power:GNDREF")
+		(at 78.74 119.38 0)
+		(unit 1)
+		(exclude_from_sim no)
+		(in_bom yes)
+		(on_board yes)
+		(dnp no)
+		(fields_autoplaced yes)
+		(property "Reference" "#PWR03"
+			(at 78.74 125.73 0)
+			(effects
+				(font
+					(size 1.27 1.27)
+				)
+				(hide yes)
+			)
+		)
+		(property "Value" "GND"
+			(at 78.74 124.46 0)
+			(effects
+				(font
+					(size 1.27 1.27)
+				)
+			)
+		)
+		(property "Footprint" ""
+			(at 78.74 119.38 0)
+			(effects
+				(font
+					(size 1.27 1.27)
+				)
+				(hide yes)
+			)
+		)
+		(property "Datasheet" ""
+			(at 78.74 119.38 0)
+			(effects
+				(font
+					(size 1.27 1.27)
+				)
+				(hide yes)
+			)
+		)
+		(property "Description" "Power symbol creates a global label with name \"GNDREF\" , reference supply ground"
+			(at 78.74 119.38 0)
+			(effects
+				(font
+					(size 1.27 1.27)
+				)
+				(hide yes)
+			)
+		)
+		(pin "1"
+		)
+		(instances
+			(project ""
+				(path "/1c8830c9-4fc6-4803-9490-280577e79dde"
+					(reference "#PWR03")
+					(unit 1)
+				)

Commit message: Finished PCB design...
Parts:
- added TB1: 1935174, 1935174, symbol SamacSys_Parts:1935174
- added TB2: 1935187, 1935187, symbol SamacSys_Parts:1935187
- added TB3: 1935776, 1935776, symbol SamacSys_Parts:1935776
- POT1: footprint Potentiometer_THT:Potentiometer_ACP_CA14-H2,5_Horizontal -> SamacSys_PCB_Library:1935174
Connections:
- net +120VAC/L: now also TB1.1
- net +120VAC/N: now also TB1.2
- net COM: now also TB2.3, TB2.4, TB3.2
- net GND: now also TB1.3
- net Vout: now also TB2.1, TB3.1
- net at BR1.1 (+), C1.1, IC1.3 (INPUT): now also TB2.2
Other:
- note added: "120VAC MAINS TERMINAL BLOCK"
- note added: "VOLT METER TERMINAL BLOCK"
